Commit message: imu calib

File: ros_ws/src/robot_control/urdf/robot.urdf.xacro (robot description, xacro)
@@ -1,6 +1,6 @@
 <?xml version="1.0"?>
 <robot name="cardboard_robot" xmlns:xacro="http://www.ros.org/wiki/xacro">
-  <!-- Import the gazebo_ros2 plugin and hardware interface macros -->
-  <xacro:include filename="$(find robot_control)/urdf/gazebo_ros2_control.urdf.xacro" />
+  <!-- Import the ros2_control interface macro -->
+  <xacro:include filename="$(find robot_control)/urdf/ros2_control.urdf.xacro" />
   <!-- Constants -->
   <xacro:property name="PI" value="3.14159265359" />
@@ -241,11 +241,16 @@
     <origin xyz="${imu_x_offset} 0 0" rpy="0 0 0"/>
   </joint>
-  <!-- Include Gazebo ROS2 control and plugin configurations -->
-  <xacro:gazebo_ros2_control
+  <!-- Include ROS2 control configuration for real hardware -->
+  <xacro:unibots_ros2_control
     wheel_separation="${wheel_separation}"
     wheel_radius="${wheel_radius}"
-    camera_name="realsense"
-    camera_frame="camera_optical_frame"
     left_wheel_joint="left_wheel_joint"
     right_wheel_joint="right_wheel_joint" />
+  <!-- Add ROS2 Control -->
+  <xacro:unibots_ros2_control
+    wheel_separation="${wheel_separation}"
+    wheel_radius="${wheel_radius}"
+    left_wheel_joint="left_wheel_joint"
+    right_wheel_joint="right_wheel_joint"
+  />
 </robot>

File: ros_ws/src/robot_control/urdf/ros2_control.urdf.xacro (robot description, xacro)
@@ -1,8 +1,15 @@
 <?xml version="1.0"?>
 <robot xmlns:xacro="http://www.ros.org/wiki/xacro">
-  <xacro:macro name="robot_control" params="name">
-    <ros2_control name="${name}" type="system">
+  <!--
+    This file contains the hardware interface configuration for ROS2 Control
+    Configured for real hardware with TB6612FNG motor driver
+  -->
+  <xacro:macro name="unibots_ros2_control"
+               params="wheel_separation wheel_radius
+                       left_wheel_joint right_wheel_joint">
+    <!-- ROS2 Control Configuration for Real Hardware -->
+    <ros2_control name="DiffDriveController" type="system">
       <hardware>
-        <plugin>robot_control_py/TB6612FNGHardwareInterface</plugin>
+        <plugin>robot_control/UnibotsMotorHardwareInterface</plugin>
         <param name="gpio_chip">gpiochip4</param>
         <!-- Left wheel motor pins -->
@@ -19,16 +26,20 @@
         <param name="left_reversed">true</param>
         <param name="right_reversed">false</param>
-        <!-- Maximum velocity that corresponds to 100% duty cycle -->
+        <!-- Max velocity that corresponds to 100% duty cycle -->
         <param name="max_velocity">10.0</param>
       </hardware>
-      <!-- Left wheel -->
-      <joint name="left_wheel_joint">
-        <command_interface name="velocity"/>
+      <joint name="${left_wheel_joint}">
+        <command_interface name="velocity">
+          <param name="min">-10</param>
+          <param name="max">10</param>
+        </command_interface>
         <state_interface name="position"/>
         <state_interface name="velocity"/>
       </joint>
-      <!-- Right wheel -->
-      <joint name="right_wheel_joint">
-        <command_interface name="velocity"/>
+      <joint name="${right_wheel_joint}">
+        <command_interface name="velocity">
+          <param name="min">-10</param>
+          <param name="max">10</param>
+        </command_interface>
         <state_interface name="position"/>
         <state_interface name="velocity"/>
